File: hardware/T-962/CPU.kicad_sch (KiCad schematic)
At the start: 11 parts

Commit message: fill out designators
Parts:
- gave numbers to parts that had none: 10
Changed lines of the file:
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@@
   (symbol (lib_id "Device:C") (at 209.55 144.78 0) (unit 1)
     (in_bom yes) (on_board yes) (fields_autoplaced)
-    (property "Reference" "C?" (id 0) (at 213.36 143.5099 0)
+    (property "Reference" "C14" (id 0) (at 213.36 143.5099 0)
       (effects (font (size 1.27 1.27)) (justify left))
     )
@@
   (symbol (lib_id "Device:R") (at 248.92 129.54 0) (unit 1)
     (in_bom yes) (on_board yes)
-    (property "Reference" "R?" (id 0) (at 246.38 132.08 90)
+    (property "Reference" "R1" (id 0) (at 246.38 132.08 90)
       (effects (font (size 1.27 1.27)) (justify left))
     )
@@
   (symbol (lib_id "Device:R") (at 60.96 128.27 90) (unit 1)
     (in_bom yes) (on_board yes)
-    (property "Reference" "R?" (id 0) (at 63.5 130.81 90)
+    (property "Reference" "R21" (id 0) (at 63.5 130.81 90)
       (effects (font (size 1.27 1.27)) (justify left))
     )
@@
   (symbol (lib_id "MCU_NXP_LPC:LPC2144FBD64") (at 148.59 92.71 0) (unit 1)
     (in_bom yes) (on_board yes)
-    (property "Reference" "U?" (id 0) (at 156.21 139.7 0)
+    (property "Reference" "U13" (id 0) (at 156.21 139.7 0)
       (effects (font (size 1.27 1.27)) (justify left))
     )
@@
   (symbol (lib_id "Device:LED") (at 73.66 128.27 180) (unit 1)
     (in_bom yes) (on_board yes)
-    (property "Reference" "D?" (id 0) (at 76.2 132.08 0))
+    (property "Reference" "L2" (id 0) (at 76.2 132.08 0))
     (property "Value" "LED" (id 1) (at 72.39 132.08 0))
     (property "Footprint" "" (id 2) (at 73.66 128.27 0)
@@
   (symbol (lib_id "Device:C") (at 165.1 34.29 0) (unit 1)
     (in_bom yes) (on_board yes) (fields_autoplaced)
-    (property "Reference" "C?" (id 0) (at 168.91 33.0199 0)
+    (property "Reference" "C13" (id 0) (at 168.91 33.0199 0)
       (effects (font (size 1.27 1.27)) (justify left))
     )
@@
   (symbol (lib_id "Device:Crystal_Small") (at 203.2 139.7 180) (unit 1)
     (in_bom yes) (on_board yes) (fields_autoplaced)
-    (property "Reference" "Y?" (id 0) (at 203.2 133.35 0))
+    (property "Reference" "Z1" (id 0) (at 203.2 133.35 0))
     (property "Value" "11.0592MHz" (id 1) (at 203.2 135.89 0))
     (property "Footprint" "" (id 2) (at 203.2 139.7 0)
@@
   (symbol (lib_id "Device:C") (at 196.85 144.78 0) (unit 1)
     (in_bom yes) (on_board yes) (fields_autoplaced)
-    (property "Reference" "C?" (id 0) (at 200.66 143.5099 0)
+    (property "Reference" "C15" (id 0) (at 200.66 143.5099 0)
       (effects (font (size 1.27 1.27)) (justify left))
     )
@@
   (symbol (lib_id "Device:R") (at 255.27 129.54 0) (unit 1)
     (in_bom yes) (on_board yes)
-    (property "Reference" "R?" (id 0) (at 252.73 132.08 90)
+    (property "Reference" "R27" (id 0) (at 252.73 132.08 90)
       (effects (font (size 1.27 1.27)) (justify left))
     )
@@
   (symbol (lib_id "Device:C") (at 248.92 148.59 0) (unit 1)
     (in_bom yes) (on_board yes) (fields_autoplaced)
-    (property "Reference" "C?" (id 0) (at 252.73 147.3199 0)
-      (effects (font (size 1.27 1.27)) (justify left))
-    )
+    (property "Reference" "C6" (id 0) (at 252.73 147.3199 0)
+      (effects (font (size 1.27 1.27)) (justify left))
+    )
