File: hardware/T-962/EEPROM.kicad_sch (KiCad schematic)
At the start: 3 parts

Commit message: fill out designators
Parts:
- gave numbers to parts that had none: 3
Changed lines of the file:
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@@
   (symbol (lib_id "Device:R") (at 121.92 85.09 0) (unit 1)
     (in_bom yes) (on_board yes)
-    (property "Reference" "R?" (id 0) (at 119.38 87.63 90)
+    (property "Reference" "R31" (id 0) (at 119.38 87.63 90)
       (effects (font (size 1.27 1.27)) (justify left))
     )
@@
   (symbol (lib_id "Memory_EEPROM:AT24CS02-SSHM") (at 154.94 93.98 0) (mirror y) (unit 1)
     (in_bom yes) (on_board yes) (fields_autoplaced)
-    (property "Reference" "U?" (id 0) (at 155.4606 83.82 0)
+    (property "Reference" "U3" (id 0) (at 155.4606 83.82 0)
       (effects (font (size 1.27 1.27)) (justify right))
     )
@@
   (symbol (lib_id "Device:R") (at 127 85.09 0) (unit 1)
     (in_bom yes) (on_board yes)
-    (property "Reference" "R?" (id 0) (at 124.46 87.63 90)
+    (property "Reference" "R32" (id 0) (at 124.46 87.63 90)
       (effects (font (size 1.27 1.27)) (justify left))
     )
